File: doc/hardware/kicad/Filament-Silicagel-Dryer/Filament-Silicagel-Dryer.kicad_pcb (KiCad board)
At the start: 2 copper layers, 76.2 x 72.4 mm, 14 parts, among them J1 Board-Connector 12Pin, J2 Conn_ESP32-S3, J3 MAX6675, U1 ESP32-DevKitC, U3 ADC1115_Shield

Commit message: Abschluß T9 Dokumentationen umsortierungen von Dateien ...
Parts:
- removed J3: MAX6675, Connector_PinHeader_2.54mm:PinHeader_1x06_P2.54mm_Vertical
- added J4: MAX6675_5pol, Connector_PinSocket_2.54mm:PinSocket_1x05_P2.54mm_Vertical, F.Cu at (101.6, 66.0)
- U4: renamed from U3; value ADC1115_Shield -> ADS1115_Shield
Routing:
- net GND: track 198.0 -> 0.00 mm
- net VCC: track 149.9 -> 0.00 mm
- net VDD: track 77.0 -> 0.00 mm
- net FAN230V: track 70.8 -> 0.00 mm, vias 1 -> 0
- net FAN12V: track 51.8 -> 0.00 mm, vias 1 -> 0
- net LAMP230V: track 42.6 -> 0.00 mm, vias 1 -> 0
- net TX2: track 41.3 -> 0.00 mm, vias 1 -> 0
- net HEATER: track 39.4 -> 0.00 mm, vias 1 -> 0
- net MOTOR230V: track 39.0 -> 0.00 mm, vias 1 -> 0
- net RX2: track 35.7 -> 0.00 mm
- net FAN230V_SLOW: track 35.4 -> 0.00 mm, vias 1 -> 0
- net CS: track 33.6 -> 0.00 mm
- net DOOR: track 32.4 -> 0.00 mm
- net SCK: track 30.0 -> 0.00 mm
- net SO: track 26.5 -> 0.00 mm
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- removed copper zone on B.Cu, net GND
- removed copper zone on F.Cu, net GND
